Commit message: debugn

File: mycobot_280/mycobot_280pi_gz/config/mycobot_280_pi.urdf.xacro (robot description, xacro)
@@ -2,6 +2,5 @@
 <!--
   Self-contained URDF xacro for mycobot_280_pi with Gazebo Ignition support.
-  Reproduces all links/joints from mycobot_description/urdf/mycobot_280_pi/mycobot_280_pi.urdf
-  and adds inertials (required for Gazebo physics) plus the ign_ros2_control plugin.
+  Collision geometry disabled — visuals + inertials only.
 -->
 <robot xmlns:xacro="http://www.ros.org/wiki/xacro" name="firefighter">
@@ -26,10 +25,4 @@
       <origin xyz="0.0 0 -0.03" rpy="0 0 1.5708"/>
     </visual>
-    <collision>
-      <geometry>
-        <mesh filename="package://mycobot_description/urdf/mycobot_280_pi/G_base.dae"/>
-      </geometry>
-      <origin xyz="0.0 0 -0.03" rpy="0 0 1.5708"/>
-    </collision>
     <inertial>
       <mass value="0.2"/>
@@ -45,10 +38,4 @@
       <origin xyz="0.0 0 0" rpy="0 0 0"/>
     </visual>
-    <collision>
-      <geometry>
-        <mesh filename="package://mycobot_description/urdf/mycobot_280_pi/joint1_pi.dae"/>
-      </geometry>
-      <origin xyz="0.0 0 0" rpy="0 0 0"/>
-    </collision>
     <inertial>
       <mass value="0.15"/>
@@ -64,10 +51,4 @@
       <origin xyz="0.0 0 -0.06096" rpy="0 0 -1.5708"/>
     </visual>
-    <collision>
-      <geometry>
-        <mesh filename="package://mycobot_description/urdf/mycobot_280_pi/joint2.dae"/>
-      </geometry>
-      <origin xyz="0.0 0 -0.06096" rpy="0 0 -1.5708"/>
-    </collision>
     <inertial>
       <mass value="0.1"/>
@@ -83,10 +64,4 @@
       <origin xyz="0.0 0 0.03256" rpy="0 -1.5708 0"/>
     </visual>
-    <collision>
-      <geometry>
-        <mesh filename="package://mycobot_description/urdf/mycobot_280_pi/joint3.dae"/>
-      </geometry>
-      <origin xyz="0.0 0 0.03256" rpy="0 -1.5708 0"/>
-    </collision>
     <inertial>
       <mass value="0.1"/>
@@ -102,10 +77,4 @@
       <origin xyz="0.0 0 0.03056" rpy="0 -1.5708 0"/>
     </visual>
-    <collision>
-      <geometry>
-        <mesh filename="package://mycobot_description/urdf/mycobot_280_pi/joint4.dae"/>
-      </geometry>
-      <origin xyz="0.0 0 0.03056" rpy="0 -1.5708 0"/>
-    </collision>
     <inertial>
       <mass value="0.1"/>
@@ -121,10 +90,4 @@
       <origin xyz="0.0 -0.001 -0.0345" rpy="0 -1.5708 1.5708"/>
     </visual>
-    <collision>
-      <geometry>
-        <mesh filename="package://mycobot_description/urdf/mycobot_280_pi/joint5.dae"/>
-      </geometry>
-      <origin xyz="0.0 -0.001 -0.0345" rpy="0 -1.5708 1.5708"/>
-    </collision>
     <inertial>
       <mass value="0.1"/>
@@ -140,10 +103,4 @@
       <origin xyz="0 0.00 -0.038" rpy="0 0 0"/>
     </visual>
-    <collision>
-      <geometry>
-        <mesh filename="package://mycobot_description/urdf/mycobot_280_pi/joint6.dae"/>
-      </geometry>
-      <origin xyz="0 0.00 -0.038" rpy="0 0 0"/>
-    </collision>
     <inertial>
       <mass value="0.05"/>
@@ -159,10 +116,4 @@
       <origin xyz="0.0 0 -0.012" rpy="0 0 0"/>
     </visual>
-    <collision>
-      <geometry>
-        <mesh filename="package://mycobot_description/urdf/mycobot_280_pi/joint7.dae"/>
-      </geometry>
-      <origin xyz="0.0 0 -0.012" rpy="0 0 0"/>
-    </collision>
     <inertial>
       <mass value="0.05"/>

Commit message: something

File: mycobot_280/mycobot_280pi_gz/config/mycobot_280_pi.urdf.xacro (robot description, xacro)
@@ -18,8 +18,14 @@
   </gazebo>
   <!-- ===== LINKS ===== -->
+  <link name="world"/>
+  <joint name="world_to_base" type="fixed">
+    <parent link="world"/>
+    <child link="g_base"/>
+    <origin xyz="0 0 0" rpy="0 0 0"/>
+  </joint>
   <link name="g_base">
     <visual>
       <geometry>
-        <mesh filename="package://mycobot_description/urdf/mycobot_280_pi/G_base.dae"/>
+        <mesh filename="package://mycobot_description/urdf/mycobot_280_pi/G_base.obj"/>
       </geometry>
       <origin xyz="0.0 0 -0.03" rpy="0 0 1.5708"/>
@@ -34,5 +40,5 @@
     <visual>
       <geometry>
-        <mesh filename="package://mycobot_description/urdf/mycobot_280_pi/joint1_pi.dae"/>
+        <mesh filename="package://mycobot_description/urdf/mycobot_280_pi/joint1_pi.obj"/>
       </geometry>
       <origin xyz="0.0 0 0" rpy="0 0 0"/>
@@ -47,5 +53,5 @@
     <visual>
       <geometry>
-        <mesh filename="package://mycobot_description/urdf/mycobot_280_pi/joint2.dae"/>
+        <mesh filename="package://mycobot_description/urdf/mycobot_280_pi/joint2.obj"/>
       </geometry>
       <origin xyz="0.0 0 -0.06096" rpy="0 0 -1.5708"/>
@@ -60,5 +66,5 @@
     <visual>
       <geometry>
-        <mesh filename="package://mycobot_description/urdf/mycobot_280_pi/joint3.dae"/>
+        <mesh filename="package://mycobot_description/urdf/mycobot_280_pi/joint3.obj"/>
       </geometry>
       <origin xyz="0.0 0 0.03256" rpy="0 -1.5708 0"/>
@@ -73,5 +79,5 @@
     <visual>
       <geometry>
-        <mesh filename="package://mycobot_description/urdf/mycobot_280_pi/joint4.dae"/>
+        <mesh filename="package://mycobot_description/urdf/mycobot_280_pi/joint4.obj"/>
       </geometry>
       <origin xyz="0.0 0 0.03056" rpy="0 -1.5708 0"/>
@@ -86,5 +92,5 @@
     <visual>
       <geometry>
-        <mesh filename="package://mycobot_description/urdf/mycobot_280_pi/joint5.dae"/>
+        <mesh filename="package://mycobot_description/urdf/mycobot_280_pi/joint5.obj"/>
       </geometry>
       <origin xyz="0.0 -0.001 -0.0345" rpy="0 -1.5708 1.5708"/>
@@ -99,5 +105,5 @@
     <visual>
       <geometry>
-        <mesh filename="package://mycobot_description/urdf/mycobot_280_pi/joint6.dae"/>
+        <mesh filename="package://mycobot_description/urdf/mycobot_280_pi/joint6.obj"/>
       </geometry>
       <origin xyz="0 0.00 -0.038" rpy="0 0 0"/>
@@ -112,5 +118,5 @@
     <visual>
       <geometry>
-        <mesh filename="package://mycobot_description/urdf/mycobot_280_pi/joint7.dae"/>
+        <mesh filename="package://mycobot_description/urdf/mycobot_280_pi/joint7.obj"/>
       </geometry>
       <origin xyz="0.0 0 -0.012" rpy="0 0 0"/>
